File: hardware/tonberry-pico/tonberry-pico.kicad_pcb (KiCad board)
At the start: 2 copper layers, 98 x 53.5 mm, 31 parts, among them J1 MicroSD_Breakout, J2 SparkFun I2S Audio Breakout M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, J3 RC522_Breakout, J4 Adafruit_bq25185_5V, J5 UART, J6 WS2812, J7 Buttons, J8 Conn_01x01, Q1 2N7000, Q2 2N7000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

Commit message: hardware: Add MSD-BO1 MicroSD Breakout
The original "SparkFun microSD Transflash Breakout" is not available any
more / currently. Add an additional footprint for the MSD-BO1 MicroSD
Breakout
(https://www.berrybase.de/micro-sd-card-reader-modul-mit-spi-schnittstelle-kompakt)
so that either one can be populated.

The MSD-BO1 has decoupling capacitors on board, so the fact that the
routing of the 3V3 trace does not "go through" the C1 capacitor is
ok. C1 does not need to be populated if the MSD-BO1 is used.

Signed-off-by: Matthias Blankertz <matthias@blankertz.org>
Parts:
- added J9: MSD_B01_MicroSD_Breakout, Modules:MSD_BO1_MicroSD_Breakout_1, F.Cu at (139.6, 43.8)
- J1: value MicroSD_Breakout -> Sparkfun_MicroSD_Breakout
Routing:
- net /SD_DO: track 27.4 -> 35.9 mm
- net +3V3: track 102.3 -> 108.7 mm
- net /SD_CS: track 14.0 -> 20.2 mm
- net /SD_DI: track 15.0 -> 21.2 mm
- net /SD_SCK: track 14.0 -> 19.4 mm
- net GND: vias 106 -> 102
Other:
- board text added: "MSD-BO1 MicroSD"
